File: pcbs/ac_dc.sch (EAGLE design)
At the start: 19 parts, among them IC1 317T, J1 22-27-2021-02, K1 G6K-2F

Commit message: AC/DC: Added atmega88 and power supply.
Parts:
- added C10, C9: 100n, resistor:C-EUC0805
- added C11: 10u, resistor:C-EUC1206
- added IC2: MEGA48/88/168-AU, avr-7:MEGA48/88/168-AU
- added U$1: TPS71530, ShortCircuitRobotics:TPS71530
Connections:
- removed net N$15: C8.+, IC1.VO
- new net +12V: C8.+, IC1.VO, U$1.VIN
- new net VCC: C10.1, C11.1, C9.1, IC2.AREF, IC2.AVCC, IC2.VCC@1, IC2.VCC@2, U$1.VOUT
- net GND: now also C10.2, C11.2, C9.2, IC2.AGND, IC2.GND@1, IC2.GND@2, U$1.GND
Other:
- moved on the sheet: C1, C2, C3, C4, C5, C6, C7, C8, D1, D2, D3, D4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

Commit message: Main Board: Added battery connector + mosfet switch
Parts:
- added JP1, JP4: (no value), pinhead:PINHD-1X5
- added JP2: (no value), pinhead:PINHD-1X4
- added JP5: (no value), pinhead:PINHD-1X2
- added Q1, Q2: MOSFET-NCHANNELSMD, SparkFun:MOSFET-NCHANNELSMD
- added R2, R4, R5: 100k, resistor:R-EU_R0805
- added R3, R6: 1k, resistor:R-EU_R0805
- added U$2: IRF7416, ShortCircuitRobotics:IRF7416
Connections:
- new net BATTERY_ON: R6.1
- new net CELL_0: JP4.4
- new net CELL_1: JP4.3
- new net CELL_2: JP4.2
- new net CELL_3: JP4.1, U$2.D1
- new net INPUT_SEL: R3.1
- new net N$11: JP1.3
- new net N$12: JP1.4
- new net N$14: K11.-, Q1.D
- new net N$15: Q1.G, R2.2, R3.2
- new net N$16: Q2.D, R4.1, U$2.G
- new net N$17: Q2.G, R5.1, R6.2
- new net N$7: JP1.2
- new net SPEED_REAR_IN: JP5.1
- new net SPEED_REAR_OUT: JP5.2
- net +12V: now also JP1.1, K11.+, R4.2, U$2.S1
- net GND: now also JP1.5, JP4.5, Q1.S, Q2.S, R2.1, R5.2
Other:
- note added: "1,315 Ohm"
- note added: "atmega88a-pa"
- note added: "from accumulator"
- note added: "to front light"
- note added: "to rear speed sensor"
- note added: "to tail light"
- moved on the sheet: C1, C2, C3, C4, C5, C6, C7, C8, D1, D2, D3, D4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
