File: pcbs/main_board.brd (EAGLE design)
At the start: 120 x 20 mm, 58 parts, among them IC1 317T, IC2 MEGA48/88/168-AU, J1 22-27-2021-02, K1 G6K-2F, Q1 MOSFET-NCHANNELSMD, Q2 MOSFET-NCHANNELSMD

Commit message: Main Board: Changed battery connection.
It does not make sense to disconnect the battery from the uC....
Instead it makes sense to disconnect the charging/input circuit
when the battery is full and disconnect the peripherals when it is
getting empty.
Parts:
- added C13: 100u, resistor:PANASONIC_E
Connections:
- net BATTERY_ON renamed CHARGING_ON
- removed net CELL3: R15.1
- removed net CELL_3: JP4.1, U$2.5, U$2.6, U$2.7, U$2.8
- new net N$23: Q2.2, R5.2
- new net N$24: C8.+, IC1.2, R4.2, U$2.1, U$2.2, U$2.3
- net +12V: now also C13.+, JP4.1, U$2.5, U$2.6, U$2.7, U$2.8; no longer C8.+, IC1.2, R4.2, U$2.1, U$2.2, U$2.3
- net GND: now also C13.-; no longer Q2.2, R5.2
Routing:
- net N$24: track 0.00 -> 13.4 mm
- net +12V: track 13.4 -> 0.00 mm
Changed lines of the file:
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@@
 <element name="R22" library="resistor" package="R0805" value="4.7k" x="-55.245" y="-227.965"/>
 <element name="R23" library="resistor" package="R0805" value="4,7k" x="-55.245" y="-233.68"/>
+<element name="C13" library="resistor" package="PANASONIC_E" value="100u" x="-52.07" y="-240.665"/>
 </elements>
 <signals>
@@
 <contactref element="R2" pad="1"/>
 <contactref element="JP4" pad="5"/>
-<contactref element="Q2" pad="2"/>
-<contactref element="R5" pad="2"/>
 <contactref element="U$3" pad="1"/>
 <contactref element="U$3" pad="3"/>
@@
 <contactref element="U$4" pad="3"/>
 <contactref element="R20" pad="2"/>
+<contactref element="C13" pad="-"/>
 <wire x1="-54.395" y1="-179.705" x2="-54.395" y2="-191.135" width="0" layer="19" extent="1-1"/>
 <wire x1="-54.395" y1="-168.275" x2="-54.395" y2="-179.705" width="0" layer="19" extent="1-1"/>
@@
 <wire x1="-44.45" y1="-116.84" x2="-44.87" y2="-120.65" width="0" layer="19" extent="1-1"/>
 <wire x1="-46.99" y1="-116.84" x2="-44.45" y2="-116.84" width="0" layer="19" extent="1-1"/>
-<wire x1="-44.87" y1="-100.33" x2="-44.45" y2="-116.84" width="0" layer="19" extent="1-1"/>
-<wire x1="-46.04" y1="-94.98" x2="-44.87" y2="-100.33" width="0" layer="19" extent="1-1"/>
 <wire x1="-54.395" y1="-208.28" x2="-54.395" y2="-191.135" width="0" layer="19" extent="1-1"/>
 <wire x1="-53.975" y1="-224.155" x2="-54.395" y2="-208.28" width="0" layer="19" extent="1-1"/>
 <wire x1="-55.245" y1="-224.155" x2="-53.975" y2="-224.155" width="0" layer="19" extent="1-1"/>
 <wire x1="-56.515" y1="-224.155" x2="-55.245" y2="-224.155" width="0" layer="19" extent="1-1"/>
-<wire x1="-31.75" y1="-67.31" x2="-46.04" y2="-94.98" width="0" layer="19" extent="1-1"/>
+<wire x1="-55.07" y1="-240.665" x2="-55.245" y2="-224.155" width="0" layer="19" extent="1-1"/>
+<wire x1="-31.75" y1="-67.31" x2="-44.45" y2="-116.84" width="0" layer="19" extent="1-1"/>
 <wire x1="-42.76" y1="-57.15" x2="-31.75" y2="-67.31" width="0" layer="19" extent="1-1"/>
 <wire x1="-35.43" y1="-31.75" x2="-42.76" y2="-57.15" width="0" layer="19" extent="1-1"/>
@@
 </signal>
 <signal name="+12V">
-<contactref element="IC1" pad="2"/>
-<contactref element="C8" pad="+"/>
-<wire x1="87.63" y1="2.54" x2="87.63" y2="5.08" width="0.8128" layer="1"/>
-<wire x1="87.63" y1="5.08" x2="88.9" y2="6.35" width="0.8128" layer="1"/>
-<wire x1="88.9" y1="6.35" x2="97.33" y2="6.35" width="0.8128" layer="1"/>
-<wire x1="97.33" y1="6.35" x2="97.79" y2="5.89" width="0.8128" layer="1"/>
 <contactref element="U$1" pad="4"/>
 <contactref element="K1" pad="1"/>
 <contactref element="JP1" pad="1"/>
-<contactref element="U$2" pad="2"/>
-<contactref element="U$2" pad="1"/>
-<contactref element="U$2" pad="3"/>
-<contactref element="R4" pad="2"/>
 <contactref element="JP2" pad="1"/>
 <contactref element="R13" pad="1"/>
 <contactref element="JP6" pad="1"/>
+<contactref element="JP4" pad="1"/>
+<contactref element="U$2" pad="5"/>
+<contactref element="U$2" pad="8"/>
+<contactref element="U$2" pad="7"/>
+<contactref element="U$2" pad="6"/>
+<contactref element="C13" pad="+"/>
 <wire x1="-55.245" y1="-203.2" x2="-56.095" y2="-162.56" width="0" layer="19" extent="1-1"/>
-<wire x1="-41.06" y1="-93.98" x2="-56.095" y2="-162.56" width="0" layer="19" extent="1-1"/>
-<wire x1="-40.64" y1="-90.17" x2="-41.06" y2="-93.98" width="0" layer="19" extent="1-1"/>
-<wire x1="-41.91" y1="-90.17" x2="-40.64" y2="-90.17" width="0" layer="19" extent="1-1"/>
-<wire x1="-43.18" y1="-90.17" x2="-41.91" y2="-90.17" width="0" layer="19" extent="1-1"/>
-<wire x1="-41.91" y1="-80.01" x2="-41.91" y2="-90.17" width="0" layer="19" extent="1-1"/>
-<wire x1="-38.1" y1="-45.72" x2="-41.91" y2="-80.01" width="0" layer="19" extent="1-1"/>
+<wire x1="-49.07" y1="-240.665" x2="-55.245" y2="-203.2" width="0" layer="19" extent="1-1"/>
+<wire x1="-43.18" y1="-83.82" x2="-56.095" y2="-162.56" width="0" layer="19" extent="1-1"/>
+<wire x1="-41.91" y1="-83.82" x2="-43.18" y2="-83.82" width="0" layer="19" extent="1-1"/>
+<wire x1="-40.64" y1="-83.82" x2="-41.91" y2="-83.82" width="0" layer="19" extent="1-1"/>
+<wire x1="-39.37" y1="-83.82" x2="-40.64" y2="-83.82" width="0" layer="19" extent="1-1"/>
+<wire x1="-41.91" y1="-80.01" x2="-41.91" y2="-83.82" width="0" layer="19" extent="1-1"/>
+<wire x1="-41.91" y1="-67.31" x2="-41.91" y2="-80.01" width="0" layer="19" extent="1-1"/>
+<wire x1="-38.1" y1="-45.72" x2="-41.91" y2="-67.31" width="0" layer="19" extent="1-1"/>
 <wire x1="-37.15" y1="-13.94" x2="-38.1" y2="-45.72" width="0" layer="19" extent="1-1"/>
 <wire x1="5.08" y1="1.48" x2="-37.15" y2="-13.94" width="0" layer="19" extent="1-1"/>
-<wire x1="87.63" y1="2.54" x2="5.08" y2="1.48" width="0" layer="19" extent="1-1"/>
 </signal>
 <signal name="N$14">
@@
 <wire x1="-56.095" y1="-227.965" x2="-34.29" y2="-80.01" width="0" layer="19" extent="1-1"/>
 </signal>
-<signal name="CELL_3">
-<contactref element="JP4" pad="1"/>
-<contactref element="U$2" pad="6"/>
-<contactref element="U$2" pad="5"/>
-<contactref element="U$2" pad="7"/>
-<contactref element="U$2" pad="8"/>
-<wire x1="-41.91" y1="-83.82" x2="-43.18" y2="-83.82" width="0" layer="19" extent="1-1"/>
-<wire x1="-40.64" y1="-83.82" x2="-41.91" y2="-83.82" width="0" layer="19" extent="1-1"/>
-<wire x1="-39.37" y1="-83.82" x2="-40.64" y2="-83.82" width="0" layer="19" extent="1-1"/>
-<wire x1="-41.91" y1="-67.31" x2="-41.91" y2="-83.82" width="0" layer="19" extent="1-1"/>
-</signal>
 <signal name="N$16">
 <contactref element="R4" pad="1"/>
@@
 <wire x1="-47.94" y1="-94.98" x2="-46.57" y2="-100.33" width="0" layer="19" extent="1-1"/>
 </signal>
-<signal name="BATTERY_ON">
+<signal name="CHARGING_ON">
 <contactref element="R6" pad="1"/>
 <contactref element="IC2" pad="8"/>
@@
 <wire x1="-24.67" y1="-0.7874" x2="-54.395" y2="-185.42" width="0" layer="19" extent="1-1"/>
 </signal>
-<signal name="CELL3">
-<contactref element="R15" pad="1"/>
-</signal>
 <signal name="N$5">
 <contactref element="JP6" pad="2"/>
@@
 <wire x1="-56.095" y1="-213.995" x2="-27.87" y2="-9.3726" width="0" layer="19" extent="1-1"/>
 </signal>
+<signal name="N$23">
+<contactref element="Q2" pad="2"/>
+<contactref element="R5" pad="2"/>
+<wire x1="-46.04" y1="-94.98" x2="-44.87" y2="-100.33" width="0" layer="19" extent="1-1"/>
+</signal>
+<signal name="N$24">
+<contactref element="IC1" pad="2"/>
+<contactref element="C8" pad="+"/>
+<wire x1="87.63" y1="2.54" x2="87.63" y2="5.08" width="0.8128" layer="1"/>
+<wire x1="87.63" y1="5.08" x2="88.9" y2="6.35" width="0.8128" layer="1"/>
+<wire x1="88.9" y1="6.35" x2="97.33" y2="6.35" width="0.8128" layer="1"/>
+<wire x1="97.33" y1="6.35" x2="97.79" y2="5.89" width="0.8128" layer="1"/>
+<contactref element="U$2" pad="2"/>
+<contactref element="U$2" pad="1"/>
+<contactref element="U$2" pad="3"/>
+<contactref element="R4" pad="2"/>
+<wire x1="-40.64" y1="-90.17" x2="-41.06" y2="-93.98" width="0" layer="19" extent="1-1"/>
+<wire x1="-41.91" y1="-90.17" x2="-40.64" y2="-90.17" width="0" layer="19" extent="1-1"/>
+<wire x1="-43.18" y1="-90.17" x2="-41.91" y2="-90.17" width="0" layer="19" extent="1-1"/>
+<wire x1="87.63" y1="2.54" x2="-40.64" y2="-90.17" width="0" layer="19" extent="1-1"/>
+</signal>
 </signals>

Commit message: Main Board: Added back i2c
Parts:
- added JP7: (no value), pinhead:1X05
- added R24: 100k, resistor:R0805
- added R25: 1k, resistor:R0805
- U$4: value IRF7413 -> IRF7103; device ShortCircuitRobotics:SO8-2 -> irf-2:SO8-2
- moved U$4 27.9 mm to (-54.0, -249.6)
Connections:
- removed net FRONT_SCL: IC2.28, JP1.4, R22.1
- removed net FRONT_SDA: IC2.27, JP1.3, R23.1
- new net BACK_I2C_POWER: R25.1
- new net N$25: JP7.5, U$4.5, U$4.6
- new net N$29: R24.1, R25.2, U$4.4
- new net SCL: IC2.28, JP1.4, JP7.4, R22.1
- new net SDA: IC2.27, JP1.3, JP7.3, R23.1
- net +12V: now also JP7.1
- net GND: now also R24.2; no longer U$4.2
- net N$22: now also U$4.2; no longer U$4.4
- net N$5: no longer U$4.5, U$4.6
- net VCC: now also JP7.2
Changed lines of the file:
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@@
 <element name="R20" library="resistor" package="R0805" value="100k" x="-55.245" y="-208.28"/>
 <element name="R21" library="resistor" package="R0805" value="1k" x="-55.245" y="-213.995"/>
-<element name="U$4" library="ShortCircuitRobotics" package="SO8-2" value="IRF7413" x="-53.975" y="-221.615"/>
 <element name="R22" library="resistor" package="R0805" value="4.7k" x="-55.245" y="-227.965"/>
 <element name="R23" library="resistor" package="R0805" value="4,7k" x="-55.245" y="-233.68"/>
 <element name="C13" library="resistor" package="PANASONIC_E" value="100u" x="-52.07" y="-240.665"/>
+<element name="U$4" library="irf-2" package="SO8-2" value="IRF7103" x="-53.975" y="-249.555"/>
+<element name="JP7" library="pinhead" package="1X05" value="" x="-50.165" y="-264.795"/>
+<element name="R24" library="resistor" package="R0805" value="100k" x="-55.245" y="-269.875"/>
+<element name="R25" library="resistor" package="R0805" value="1k" x="-55.245" y="-275.59"/>
 </elements>
 <signals>
@@
 <contactref element="R16" pad="2"/>
 <contactref element="R18" pad="2"/>
-<contactref element="U$4" pad="2"/>
-<contactref element="U$4" pad="1"/>
-<contactref element="U$4" pad="3"/>
 <contactref element="R20" pad="2"/>
 <contactref element="C13" pad="-"/>
+<contactref element="U$4" pad="1"/>
+<contactref element="R24" pad="2"/>
+<contactref element="U$4" pad="3"/>
 <wire x1="-54.395" y1="-179.705" x2="-54.395" y2="-191.135" width="0" layer="19" extent="1-1"/>
 <wire x1="-54.395" y1="-168.275" x2="-54.395" y2="-179.705" width="0" layer="19" extent="1-1"/>
@@
 <wire x1="-46.99" y1="-116.84" x2="-44.45" y2="-116.84" width="0" layer="19" extent="1-1"/>
 <wire x1="-54.395" y1="-208.28" x2="-54.395" y2="-191.135" width="0" layer="19" extent="1-1"/>
-<wire x1="-53.975" y1="-224.155" x2="-54.395" y2="-208.28" width="0" layer="19" extent="1-1"/>
-<wire x1="-55.245" y1="-224.155" x2="-53.975" y2="-224.155" width="0" layer="19" extent="1-1"/>
-<wire x1="-56.515" y1="-224.155" x2="-55.245" y2="-224.155" width="0" layer="19" extent="1-1"/>
-<wire x1="-55.07" y1="-240.665" x2="-55.245" y2="-224.155" width="0" layer="19" extent="1-1"/>
+<wire x1="-55.07" y1="-240.665" x2="-54.395" y2="-208.28" width="0" layer="19" extent="1-1"/>
+<wire x1="-53.975" y1="-252.095" x2="-55.07" y2="-240.665" width="0" layer="19" extent="1-1"/>
+<wire x1="-56.515" y1="-252.095" x2="-53.975" y2="-252.095" width="0" layer="19" extent="1-1"/>
+<wire x1="-54.395" y1="-269.875" x2="-53.975" y2="-252.095" width="0" layer="19" extent="1-1"/>
 <wire x1="-31.75" y1="-67.31" x2="-44.45" y2="-116.84" width="0" layer="19" extent="1-1"/>
 <wire x1="-42.76" y1="-57.15" x2="-31.75" y2="-67.31" width="0" layer="19" extent="1-1"/>
@@
 <contactref element="R22" pad="2"/>
 <contactref element="R23" pad="2"/>
+<contactref element="JP7" pad="2"/>
 <wire x1="-54.395" y1="-227.965" x2="-56.095" y2="-196.85" width="0" layer="19" extent="1-1"/>
 <wire x1="-54.395" y1="-233.68" x2="-54.395" y2="-227.965" width="0" layer="19" extent="1-1"/>
+<wire x1="-52.705" y1="-264.795" x2="-54.395" y2="-233.68" width="0" layer="19" extent="1-1"/>
 <wire x1="-55.88" y1="-135.89" x2="-56.095" y2="-196.85" width="0" layer="19" extent="1-1"/>
 <wire x1="-39.37" y1="-80.01" x2="-55.88" y2="-135.89" width="0" layer="19" extent="1-1"/>
@@
 <contactref element="U$2" pad="6"/>
 <contactref element="C13" pad="+"/>
+<contactref element="JP7" pad="1"/>
 <wire x1="-55.245" y1="-203.2" x2="-56.095" y2="-162.56" width="0" layer="19" extent="1-1"/>
 <wire x1="-49.07" y1="-240.665" x2="-55.245" y2="-203.2" width="0" layer="19" extent="1-1"/>
+<wire x1="-55.245" y1="-264.795" x2="-49.07" y2="-240.665" width="0" layer="19" extent="1-1"/>
 <wire x1="-43.18" y1="-83.82" x2="-56.095" y2="-162.56" width="0" layer="19" extent="1-1"/>
 <wire x1="-41.91" y1="-83.82" x2="-43.18" y2="-83.82" width="0" layer="19" extent="1-1"/>
@@
 <wire x1="-30.9626" y1="-3.08" x2="-39.37" y2="-73.66" width="0" layer="19" extent="1-1"/>
 </signal>
-<signal name="FRONT_SDA">
+<signal name="SDA">
 <contactref element="JP1" pad="3"/>
 <contactref element="IC2" pad="27"/>
 <contactref element="R23" pad="1"/>
+<contactref element="JP7" pad="3"/>
 <wire x1="-25.47" y1="-0.7874" x2="-36.83" y2="-80.01" width="0" layer="19" extent="1-1"/>
 <wire x1="-56.095" y1="-233.68" x2="-36.83" y2="-80.01" width="0" layer="19" extent="1-1"/>
-</signal>
-<signal name="FRONT_SCL">
+<wire x1="-50.165" y1="-264.795" x2="-56.095" y2="-233.68" width="0" layer="19" extent="1-1"/>
+</signal>
+<signal name="SCL">
 <contactref element="JP1" pad="4"/>
 <contactref element="IC2" pad="28"/>
 <contactref element="R22" pad="1"/>
+<contactref element="JP7" pad="4"/>
 <wire x1="-26.27" y1="-0.7874" x2="-34.29" y2="-80.01" width="0" layer="19" extent="1-1"/>
 <wire x1="-56.095" y1="-227.965" x2="-34.29" y2="-80.01" width="0" layer="19" extent="1-1"/>
+<wire x1="-47.625" y1="-264.795" x2="-56.095" y2="-227.965" width="0" layer="19" extent="1-1"/>
 </signal>
 <signal name="N$16">
@@
 <signal name="N$5">
 <contactref element="JP6" pad="2"/>
-<contactref element="U$4" pad="6"/>
-<contactref element="U$4" pad="5"/>
 <contactref element="U$4" pad="8"/>
 <contactref element="U$4" pad="7"/>
-<wire x1="-55.245" y1="-217.805" x2="-56.515" y2="-217.805" width="0" layer="19" extent="1-1"/>
-<wire x1="-53.975" y1="-217.805" x2="-55.245" y2="-217.805" width="0" layer="19" extent="1-1"/>
-<wire x1="-52.705" y1="-217.805" x2="-53.975" y2="-217.805" width="0" layer="19" extent="1-1"/>
-<wire x1="-52.705" y1="-203.2" x2="-52.705" y2="-217.805" width="0" layer="19" extent="1-1"/>
+<wire x1="-55.245" y1="-245.745" x2="-56.515" y2="-245.745" width="0" layer="19" extent="1-1"/>
+<wire x1="-52.705" y1="-203.2" x2="-55.245" y2="-245.745" width="0" layer="19" extent="1-1"/>
 </signal>
 <signal name="N$22">
 <contactref element="R21" pad="2"/>
 <contactref element="R20" pad="1"/>
-<contactref element="U$4" pad="4"/>
-<wire x1="-54.395" y1="-213.995" x2="-52.705" y2="-224.155" width="0" layer="19" extent="1-1"/>
+<contactref element="U$4" pad="2"/>
+<wire x1="-54.395" y1="-213.995" x2="-55.245" y2="-252.095" width="0" layer="19" extent="1-1"/>
 <wire x1="-56.095" y1="-208.28" x2="-54.395" y2="-213.995" width="0" layer="19" extent="1-1"/>
 </signal>
@@
 <wire x1="87.63" y1="2.54" x2="-40.64" y2="-90.17" width="0" layer="19" extent="1-1"/>
 </signal>
+<signal name="N$25">
+<contactref element="JP7" pad="5"/>
+<contactref element="U$4" pad="6"/>
+<contactref element="U$4" pad="5"/>
+<wire x1="-52.705" y1="-245.745" x2="-45.085" y2="-264.795" width="0" layer="19" extent="1-1"/>
+<wire x1="-53.975" y1="-245.745" x2="-52.705" y2="-245.745" width="0" layer="19" extent="1-1"/>
+</signal>
+<signal name="N$29">
+<contactref element="R25" pad="2"/>
+<contactref element="R24" pad="1"/>
+<contactref element="U$4" pad="4"/>
+<wire x1="-56.095" y1="-269.875" x2="-54.395" y2="-275.59" width="0" layer="19" extent="1-1"/>
+<wire x1="-52.705" y1="-252.095" x2="-56.095" y2="-269.875" width="0" layer="19" extent="1-1"/>
+</signal>
+<signal name="BACK_I2C_POWER">
+<contactref element="R25" pad="1"/>
+</signal>
 </signals>
