File: pcbs/main_board.brd (EAGLE design)
At the start: 120 x 20 mm, 62 parts, among them IC1 317T, IC2 MEGA48/88/168-AU, J1 22-27-2021-02, K1 G6K-2F, Q1 MOSFET-NCHANNELSMD, Q2 MOSFET-NCHANNELSMD

Commit message: Main Board: Started layouting control part
Parts:
- removed JP1, JP4, JP7: (no value), pinhead:1X05
- removed JP2: (no value), pinhead:1X04
- removed JP5, JP6: (no value), pinhead:1X02
- added 12V, REAR_SPEED: (no value), pinhead:1X02
- added BACK_I2C, BAT, FRONT_LIGHT: (no value), pinhead:1X05
- added TAIL_LIGH: (no value), pinhead:1X04
- moved R25 329.5 mm to (75.7, 26.8)
- moved R24 326.4 mm to (80.5, 26.9), turned to 90 degrees
- moved C13 318.6 mm to (87.6, 45.7)
- moved U$4 308.9 mm to (86.0, 25.8), turned to 270 degrees
- moved R20 276.1 mm to (84.3, 30.0)
- moved R21 275.8 mm to (75.7, 28.7)
- moved R18 274.1 mm to (63.1, 56.1)
- moved R23 269.8 mm to (28.2, 22.9), turned to 270 degrees
- moved R22 265.0 mm to (30.2, 22.9), turned to 270 degrees
- moved R17 260.3 mm to (54.9, 50.4)
- moved R13 251.7 mm to (73.0, 54.0)
- moved R16 248.5 mm to (54.2, 43.4)
- moved R14 244.7 mm to (61.8, 46.6)
- moved R12 242.9 mm to (74.2, 48.8)
- moved R15 241.5 mm to (47.2, 44.7)
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Connections:
- net +12V: now also 12V.1, BACK_I2C.1, BAT.1, FRONT_LIGHT.1, TAIL_LIGH.1; no longer JP1.1, JP2.1, JP4.1, JP6.1, JP7.1
- net CELL_0: now also BAT.4; no longer JP4.4
- net CELL_1: now also BAT.3; no longer JP4.3
- net CELL_2: now also BAT.2; no longer JP4.2
- net GND: now also BAT.5; no longer JP4.5
- net N$13: now also FRONT_LIGHT.5; no longer JP1.5
- net N$18: now also TAIL_LIGH.3; no longer JP2.3
- net N$25: now also BACK_I2C.5; no longer JP7.5
- net N$5: now also 12V.2; no longer JP6.2
- net SCL: now also BACK_I2C.4, FRONT_LIGHT.4; no longer JP1.4, JP7.4
- net SDA: now also BACK_I2C.3, FRONT_LIGHT.3; no longer JP1.3, JP7.3
- net SPEED_REAR_IN: now also REAR_SPEED.1; no longer JP5.1
- net SPEED_REAR_OUT: now also REAR_SPEED.2; no longer JP5.2
- net TAIL_LIGHT: now also TAIL_LIGH.2; no longer JP2.2
- net TAIL_PWM: now also TAIL_LIGH.4; no longer JP2.4
- net VCC: now also BACK_I2C.2, FRONT_LIGHT.2; no longer JP1.2, JP7.2
Routing:
- net +12V: track 0.00 -> 18.1 mm
- net GND: track 68.1 -> 83.4 mm
- net N$24: track 13.4 -> 28.5 mm
- net N$25: track 0.00 -> 11.4 mm
- net N$5: track 0.00 -> 9.18 mm
- net N$16: track 0.00 -> 7.69 mm
- net VCC: track 0.00 -> 5.42 mm
- net N$22: track 0.00 -> 5.08 mm
- net N$17: track 0.00 -> 4.20 mm
- net N$23: track 0.00 -> 1.84 mm
Other:
- board size 120 x 20 mm -> 100 x 40 mm
