File: pcbs/main_board.brd (EAGLE design)
At the start: 100 x 40 mm, 62 parts, among them IC1 317T, IC2 MEGA48/88/168-AU, J1 22-27-2021-02, K1 G6K-2F, Q1 MOSFET-NCHANNELSMD, Q2 MOSFET-NCHANNELSMD

Commit message: Pcbs: latest changes
Parts:
- removed BACK_I2C, BAT, FRONT_LIGHT: (no value), pinhead:1X05
- removed C1, C2: 82µ, resistor:175TMP-0808
- removed D4: (no value), diode:DO-214AC
- removed J1: 22-27-2021-02, con-molex:6410-02
- removed JP3: AVR-ISP-6VERT, ShortCircuitRobotics:AVR-ISP-6
- removed K1: G6K-2F, relay:G6K-2F
- removed Q1: MOSFET-NCHANNELSMD, SparkFun:SOT23-3
- removed R1: (no value), resistor:R1206
- removed R2, R24: 100k, resistor:R0805
- removed R25, R3: 1k, resistor:R0805
- added BAT_+, BAT_-, BAT_0, BAT_1, BAT_2, GENERATOR_+, GENERATOR_-: TPTP18SQ, testpad:TP18SQ
- added U$5: ISP_SPECIALS, bookla:ISP_RM2_00_STRAIGHT
- C3, C4: value 82µ -> 220u; device resistor:175TMP-0808 -> resistor:PANASONIC_F
- D6: value (none) -> 2.7V
- R10, R21, R6, R9: value 1k -> 33; device resistor:R0805 -> resistor:R0603
- R11, R12, R13, R14, R15, R16, R17, R18, R19, R20, R22, R23, R4, R5, R7, R8: device resistor:R0805 -> resistor:R0603
- moved 12V 164.9 mm to (-69.8, 50.8), turned to 0 degrees
- moved U$1 143.9 mm to (-63.4, 35.6)
- moved U$4 138.3 mm to (-52.0, 35.6), turned to 0 degrees
- moved R20 135.3 mm to (-48.2, 57.2)
- moved C11 125.9 mm to (-48.2, 44.4), turned to 0 degrees
- moved R17 125.3 mm to (-69.8, 63.4)
- moved R13 123.0 mm to (-49.6, 63.4)
- moved C9 121.6 mm to (-67.4, 57.2), turned to 0 degrees
- moved R16 120.7 mm to (-64.8, 63.4)
- moved R12 119.5 mm to (-44.4, 63.4)
- moved R14 117.7 mm to (-54.6, 63.4)
- moved R11 108.7 mm to (-39.4, 63.4)
- moved R15 108.5 mm to (-59.6, 63.4)
- moved IC2 106.9 mm to (-66.0, 5.00)
- moved R21 105.6 mm to (-21.6, 69.8)
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Connections:
- removed net BACK_I2C_POWER: R25.1
- removed net INPUT_SEL: IC2.7, R3.1
- removed net N$11: C2.-, D3.C, D4.A
- removed net N$14: K1.8, Q1.3
- removed net N$15: Q1.1, R2.2, R3.2
- removed net N$23: Q2.2, R5.2
- removed net N$25: BACK_I2C.5, U$4.5, U$4.6
- removed net N$29: R24.1, R25.2, U$4.4
- removed net N$3: C1.+, C2.+, R1.1
- removed net N$6: C1.-, K1.4, K1.5
- net +12V: now also BAT_+.TP; no longer BACK_I2C.1, BAT.1, FRONT_LIGHT.1, K1.1
- net CELL_0: now also BAT_0.TP; no longer BAT.4
- net CELL_1: now also BAT_1.TP; no longer BAT.3
- net CELL_2: now also BAT_2.TP; no longer BAT.2
- net GND: now also BAT_-.TP, C7.2, C8.-, Q2.2, R5.2, U$5.VCC; no longer BAT.5, D3.A, JP3.6, Q1.2, R2.1, R24.2, U$4.3
- net N$1: now also D3.C, R4.2, U$2.1, U$2.2, U$2.3; no longer C3.-, C4.+, K1.2, K1.7
- net N$10: no longer C7.2, C8.-
- net N$12: now also U$5.RESET; no longer JP3.1
- net N$13: no longer FRONT_LIGHT.5
- net N$21: now also U$5.MOSI; no longer JP3.4
- net N$24: now also D3.A; no longer R4.2, U$2.1, U$2.2, U$2.3
- net N$4: now also GENERATOR_-.TP; no longer J1.2
- net N$7: now also U$5.SCK; no longer JP3.3
- net N$8: now also C3.-, C4.+; no longer K1.3, K1.6
- net N$9: now also GENERATOR_+.TP; no longer J1.1
- net RESET: now also U$5.MISO; no longer JP3.5
- net SCL: no longer BACK_I2C.4, FRONT_LIGHT.4
- net SDA: no longer BACK_I2C.3, FRONT_LIGHT.3
- net VCC: now also U$5.GND; no longer BACK_I2C.2, FRONT_LIGHT.2, JP3.2
- net V_IN: no longer D4.C, R1.2
Routing:
- net V_IN: track 127.2 -> 69.7 mm
- net N$11: track 39.3 -> 0.00 mm
- net GND: track 83.4 -> 121.9 mm
- net N$6: track 36.5 -> 0.00 mm
- net N$3: track 17.8 -> 0.00 mm
- net N$10: track 28.9 -> 13.0 mm, vias 0 -> 1
- net N$24: track 28.5 -> 12.8 mm
- net N$25: track 11.4 -> 0.00 mm
- net N$5: track 9.18 -> 0.00 mm
- net N$9: track 0.00 -> 8.15 mm
- net N$16: track 7.69 -> 13.7 mm
- net VCC: track 5.42 -> 0.00 mm
- net +12V: track 18.1 -> 23.4 mm
- net N$22: track 5.08 -> 0.00 mm
- net N$8: track 15.6 -> 11.2 mm
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Other:
- board size 100 x 40 mm -> 70 x 20 mm
