File: pcbs/front_light.brd (EAGLE design)
At the start: 32.5 x 25.2 mm, 44 parts, among them IC1 LT3474, IC3 ATTINY24/44/84-SSU, Q1 BSS123

Commit message: Pcbs: latest changes
Parts:
- removed LOGO1: OSHW_LOGO_6MILX0070-NT, ea:OSHW_6X70_NOTEXT
- added LOGO2: OSHW_LOGO_6MILX0150-NT, ea:OSHW_6X150_NOTEXT
- moved C14 5.75 mm to (8.25, 2.00)
- renumbered IC1 to LT3474, IC3 to ATTINY24
Routing:
- net VCC: track 35.8 -> 39.5 mm
Other:
- board text added: "(C) eKiwi 2013"
- board text added: "+12V"
- board text added: "Big"
- board text added: "DLR"
- board text added: "GND"
- board text added: "IN"
- board text added: "OUT"
- board text added: "WAKE"
- board text added: "licensed under CERN OHL v1.2"
- board text removed: "eKiwi"
