File: pcbs/main_board.sch (EAGLE design)
At the start: 62 parts, among them IC1 317T, IC2 MEGA48/88/168-AU, J1 22-27-2021-02, K1 G6K-2F, Q1 MOSFET-NCHANNELSMD, Q2 MOSFET-NCHANNELSMD

Commit message: Pcbs: latest changes
Parts:
- removed BACK_I2C, BAT, FRONT_LIGHT: (no value), pinhead:PINHD-1X5
- removed C1, C2: 82µ, resistor:CPOL-EU175TMP-0808
- removed D4: (no value), diode:DIODE-DO-214AC
- removed J1: 22-27-2021-02, con-molex:22-27-2021-02
- removed JP3: AVR-ISP-6VERT, ShortCircuitRobotics:AVR-ISP-6VERT
- removed K1: G6K-2F, relay:G6K-2F
- removed Q1: MOSFET-NCHANNELSMD, SparkFun:MOSFET-NCHANNELSMD
- removed R1: (no value), resistor:R-EU_R1206
- removed R2, R24: 100k, resistor:R-EU_R0805
- removed R25, R3: 1k, resistor:R-EU_R0805
- added BAT_+, BAT_-, BAT_0, BAT_1, BAT_2, GENERATOR_+, GENERATOR_-: TPTP18SQ, testpad:TPTP18SQ
- added U$5: ISP_SPECIALS, bookla:ISP_SPECIALS
- C3, C4: value 82µ -> 220u; device resistor:CPOL-EU175TMP-0808 -> resistor:CPOL-EUF
- D6: value (none) -> 2.7V
- R10, R21, R6, R9: value 1k -> 33; device resistor:R-EU_R0805 -> resistor:R-EU_R0603
- R11, R12, R13, R14, R15, R16, R17, R18, R19, R20, R22, R23, R4, R5, R7, R8: device resistor:R-EU_R0805 -> resistor:R-EU_R0603
Connections:
- removed net BACK_I2C_POWER: R25.1
- removed net INPUT_SEL: IC2.PB6(XTAL1/TOSC1/PCINT6), R3.1
- removed net N$11: C2.-, D3.C, D4.A
- removed net N$14: K11.-, Q1.D
- removed net N$15: Q1.G, R2.2, R3.2
- removed net N$23: Q2.S, R5.2
- removed net N$25: BACK_I2C.5, U$4G$2.D@1, U$4G$2.D@2
- removed net N$29: R24.1, R25.2, U$4G$2.G
- removed net N$3: C1.+, C2.+, R1.1
- removed net N$6: C1.-, K12.S, K13.S
- net +12V: now also BAT_+.TP; no longer BACK_I2C.1, BAT.1, FRONT_LIGHT.1, K11.+
- net CELL_0: now also BAT_0.TP; no longer BAT.4
- net CELL_1: now also BAT_1.TP; no longer BAT.3
- net CELL_2: now also BAT_2.TP; no longer BAT.2
- net GND: now also BAT_-.TP, C7.2, C8.-, Q2.S, R5.2, U$5.GND; no longer BAT.5, D3.A, JP3.6, Q1.S, R2.1, R24.2, U$4G$2.S
- net N$1: now also D3.C, R4.2, U$2.S1; no longer C3.-, C4.+, K12.O, K13.O
- net N$10: no longer C7.2, C8.-
- net N$12: now also U$5.MISO; no longer JP3.1
- net N$13: no longer FRONT_LIGHT.5
- net N$21: now also U$5.MOSI; no longer JP3.4
- net N$24: now also D3.A; no longer R4.2, U$2.S1
- net N$4: now also GENERATOR_-.TP; no longer J1-2.S
- net N$7: now also U$5.SCK; no longer JP3.3
- net N$8: now also C3.-, C4.+; no longer K12.P, K13.P
- net N$9: now also GENERATOR_+.TP; no longer J1-1.S
- net RESET: now also U$5.RESET; no longer JP3.5
- net SCL: no longer BACK_I2C.4, FRONT_LIGHT.4
- net SDA: no longer BACK_I2C.3, FRONT_LIGHT.3
- net VCC: now also U$5.VCC; no longer BACK_I2C.2, FRONT_LIGHT.2, JP3.2
- net V_IN: no longer D4.C, R1.2
Other:
- note added: "12V + 2.7V = 14.7V 14.7V / 4 cells = 3.675V per cell"
- note removed: "1,315 Ohm"
- note removed: "back i2c"
- moved on the sheet: C10, C11, C13, C3, C4, C5, C6, C7, C8, C9, D1, D2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
